File: DataLogger2025.kicad_pcb (KiCad board)
At the start: 2 copper layers, 80 x 80 mm, 66 parts, among them J1 2171790001, J2 2908-05WB-MG, J3 0436500201 1x02, J5 0436500201 1x02, J6 0436500201 1x02, J7 B10B-XH-A, SW1 SMD_4.6x2.8mm_h1.9mm, U2 SM24CANB-02HTG, U3 SN65HVD230, U4 ESP32-S3-WROOM-1U-N16R8

Commit message: Add files via upload
Parts:
- added C23: 100nF, Capacitor_SMD:C_1206_3216Metric_Pad1.33x1.80mm_HandSolder, B.Cu at (72.4, 79.5)
- added TP1: TestPoint, TestPoint:TestPoint_Pad_1.5x1.5mm, F.Cu at (58.5, 86.0)
- added TP2: TestPoint, TestPoint:TestPoint_Pad_1.5x1.5mm, F.Cu at (49.2, 55.7)
- added TP3: TestPoint, TestPoint:TestPoint_Pad_1.5x1.5mm, F.Cu at (64.1, 44.1)
- added TP4: TestPoint, TestPoint:TestPoint_Pad_1.5x1.5mm, F.Cu at (66.5, 89.0)
- added TP5: TestPoint, TestPoint:TestPoint_Pad_1.5x1.5mm, F.Cu at (59.5, 93.5)
- added TP6: TestPoint, TestPoint:TestPoint_Pad_1.5x1.5mm, B.Cu at (98.0, 42.0)
- added TP7: TestPoint, TestPoint:TestPoint_Pad_1.5x1.5mm, B.Cu at (93.0, 42.0)
- added TP8: TestPoint, TestPoint:TestPoint_Pad_1.0x1.0mm, F.Cu at (61.1, 36.5)
- added TP9: TestPoint, TestPoint:TestPoint_Pad_1.5x1.5mm, F.Cu at (90.5, 61.0)
- added U1: USBLC6-2SC6, USBLC6-2SC6:SOT95P280X145-6N, F.Cu at (74.0, 84.0)
- moved R5 2.48 mm to (78.5, 86.0)
Connections:
- J1 pad A6: /USB_D+ -> Net-(J1-DP1)
- J1 pad A7: /USB_D- -> Net-(J1-DN1)
- J1 pad B6: /USB_D+ -> Net-(J1-DP1)
- J1 pad B7: /USB_D- -> Net-(J1-DN1)
Routing:
- net Net-(D2-A): track 33.8 -> 50.2 mm, vias 0 -> 2
- net /USB_D-: track 51.3 -> 39.4 mm, vias 2 -> 0
- net /USB_D+: track 49.6 -> 38.3 mm, vias 0 -> 2
- net Net-(J1-DN1): track 0.00 -> 9.53 mm, vias 0 -> 3
- net Net-(J1-DP1): track 0.00 -> 9.45 mm
- net /V_Dirty_MBAT: track 15.8 -> 21.1 mm
- net /5V_CLEAN: track 28.2 -> 31.5 mm
- net /IO0_Boot: track 22.4 -> 25.5 mm
- net /3V3_CLEAN: track 172.1 -> 174.9 mm
- net /CAN_LOW: track 11.5 -> 13.9 mm
- net /CAN_HIGH: track 11.3 -> 13.8 mm
- net Net-(U4-EN): track 9.38 -> 11.0 mm
- net GND: vias 156 -> 159
Other:
- board text added: "MotoLogger Rev A 7/2026"
- board text added: "WayWayWay"
