File: DataLogger2025.kicad_sch (KiCad schematic)
At the start: 62 parts, among them J1 2171790001, J2 2908-05WB-MG, J3 0436500201 1x02, J5 0436500201 1x02, J6 0436500201 1x02, J7 B10B-XH-A, SW1 SMD_4.6x2.8mm_h1.9mm, U2 SM24CANB-02HTG, U3 SN65HVD230, U4 ESP32-S3-WROOM-1U-N16R8

Commit message: Add files via upload
Parts:
- added C23: 100nF, Capacitor_SMD:C_1206_3216Metric_Pad1.33x1.80mm_HandSolder, symbol Device:C_Small
- added TP1, TP2, TP3, TP4, TP5, TP6, TP7, TP9: TestPoint, TestPoint:TestPoint_Pad_1.5x1.5mm, symbol Connector:TestPoint
- added TP8: TestPoint, TestPoint:TestPoint_Pad_1.0x1.0mm, symbol Connector:TestPoint
- added U1: USBLC6-2SC6, USBLC6-2SC6:SOT95P280X145-6N, symbol Power_Protection:USBLC6-2SC6
Connections:
- net 3V3_CLEAN: now also TP3.1
- net 5V_CLEAN: now also TP2.1
- net CAN_HIGH: now also TP7.1
- net CAN_LOW: now also TP6.1
- net GND: now also C23.2, TP5.1, U1.2 (GND)
- net IO0_Boot: now also TP9.1
- net USB_D+: now also U1.6 (I/O1); no longer J1.A6 (DP1), J1.B6 (DP2)
- net USB_D-: now also U1.4 (I/O2); no longer J1.A7 (DN1), J1.B7 (DN2)
- net V_Dirty_MBAT: now also TP1.1
- net at C22.1, R1.2, U4.3 (EN): now also TP8.1
- net at D2.2 (A), J1.A4B9 (VBUS1), J1.B4A9 (VBUS2): now also C23.1, TP4.1, U1.5 (VBUS)
- new net: J1.A6 (DP1), J1.B6 (DP2), U1.1 (I/O1)
- new net: J1.A7 (DN1), J1.B7 (DN2), U1.3 (I/O2)
