File: Moto_PCBs/Moto_Mobo/DataLogger2025.kicad_pcb (KiCad board)
At the start: 2 copper layers, 80 x 80 mm, 77 parts, among them J1 2171790001, J2 2908-05WB-MG, J3 0436500201 1x02, J5 0436500201 1x02, J6 0436500201 1x02, J7 B10B-XH-A, SW1 SMD_4.6x2.8mm_h1.9mm, U1 USBLC6-2SC6, U2 SM24CANB-02HTG, U3 SN65HVD230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

Commit message: Final Mobo GBR/PCB Files before PCBWAY Order
Parts:
- removed C23: 100nF, Capacitor_SMD:C_1206_3216Metric_Pad1.33x1.80mm_HandSolder
- removed FL1: DLW21SZ900HQ2L, DLW21SZ900HQ2L:FIL_DLW21SZ900HQ2L
- added CR1: RCLAMP0504S.TCT, RCLAMP0504S.TCT:SC70-6L_RCLAMP_1p75x3p1-0p95_SEM, F.Cu at (70.0, 83.0)
- U1: value USBLC6-2SC6 -> DLW21SH900HQ2L; footprint USBLC6-2SC6:SOT95P280X145-6N -> DLW21SH900HQ2L:DLW21SH_MUR
- moved U1 47.4 mm to (95.2, 41.5), turned to -90 degrees
- moved R4 5.76 mm to (70.0, 78.0), turned to -90 degrees
Connections:
- J1 pad A6: Net-(J1-DP1) -> /USB_D+
- J1 pad A7: Net-(J1-DN1) -> /USB_D-
- J1 pad B6: Net-(J1-DP1) -> /USB_D+
- J1 pad B7: Net-(J1-DN1) -> /USB_D-
- J3 pad 1: Net-(FL1-Pad2) -> Net-(J3-Pad1)
- J3 pad 2: Net-(FL1-Pad3) -> Net-(J3-Pad2)
- U1 pad 1: Net-(J1-DP1) -> /CAN_LOW
- U1 pad 2: GND -> /CAN_HIGH
- U1 pad 3: Net-(J1-DN1) -> Net-(J3-Pad1)
- U1 pad 4: /USB_D- -> Net-(J3-Pad2)
- U2 pad 1: Net-(FL1-Pad2) -> Net-(J3-Pad1)
- U2 pad 2: Net-(FL1-Pad3) -> Net-(J3-Pad2)
Routing:
- net Net-(J3-Pad1): track 0.00 -> 20.6 mm
- net Net-(FL1-Pad2): track 20.6 -> 0.00 mm
- net /USB_D+: track 38.3 -> 54.9 mm
- net /USB_D-: track 39.4 -> 53.5 mm, vias 0 -> 2
- net Net-(J3-Pad2): track 0.00 -> 13.4 mm
- net Net-(FL1-Pad3): track 13.4 -> 0.00 mm
- net Net-(D2-A): track 50.2 -> 39.1 mm, vias 2 -> 0
- net Net-(J1-DN1): track 9.53 -> 0.00 mm, vias 3 -> 0
- net Net-(J1-DP1): track 9.45 -> 0.00 mm
- net Net-(J1-CC1): track 6.52 -> 12.1 mm
- net GND: vias 159 -> 163
