File: Moto_PCBs/Moto_Mobo/DataLogger2025.kicad_pcb (KiCad board)
At the start: 2 copper layers, 80 x 80 mm, 76 parts, among them J1 2171790001, J2 2908-05WB-MG, J3 0436500201 1x02, J5 0436500201 1x02, J6 0436500201 1x02, J7 B10B-XH-A, SW1 SMD_4.6x2.8mm_h1.9mm, U1 DLW21SH900HQ2L, U2 SM24CANB-02HTG, U3 SN65HVD230, U4 ESP32-S3-WROOM-1U-N16R8

Commit message: Add files via upload
Routing:
- net GND: vias 163 -> 167
Other:
- board text added: "MotoLogger Rev A 2026"
- board text added: "Night Shift Electronics"
- board text removed: "MotoLogger Rev A 7/2026"
Changed lines of the file:
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@@
 		(sheetname "/")
 		(sheetfile "DataLogger2025.kicad_sch")
-		(units
-			(unit
-				(name "A")
-				(pins "3" "36" "37" "27" "39" "38" "15" "4" "5" "6" "7" "12" "17" "18"
-					"19" "20" "21" "22" "2" "8" "9" "10" "11" "13" "14" "23" "28" "29" "30"
-					"31" "32" "33" "34" "35" "26" "16" "24" "25" "1" "40" "41_1" "41_2"
-					"41_3" "41_4" "41_5" "41_6" "41_7" "41_8" "41_9"
-				)
-			)
-		)
 		(attr smd)
 		(duplicate_pad_numbers_are_jumpers no)
@@
 		)
 		(fp_circle
-			(center -10.5 -8.41)
-			(end -10.4 -8.41)
+			(center -7.5 -8.41)
+			(end -7.4 -8.41)
 			(stroke
 				(width 0.2)
@@
 		)
 		(fp_circle
-			(center -10.5 -8.41)
-			(end -10.4 -8.41)
+			(center -7.5 -8.41)
+			(end -7.4 -8.41)
 			(stroke
 				(width 0.2)
@@
 			(pinfunction "1_1")
 			(pintype "passive")
+			(zone_connect 2)
 		)
 		(embedded_fonts no)
@@
 		)
 	)
-	(gr_text "MotoLogger Rev A 7/2026"
-		(at 80.5 97 0)
+	(gr_text "WayWayWay"
+		(at 80.5 93 0)
 		(layer "F.SilkS")
 		(effects
@@
 		)
 	)
-	(gr_text "WayWayWay"
-		(at 81.801111 95.122736 0)
+	(gr_text "MotoLogger Rev A 2026"
+		(at 80.5 95 0)
+		(layer "F.SilkS")
+		(effects
+			(font
+				(size 1 1)
+				(bold yes)
+			)
+			(justify left bottom)
+		)
+	)
+	(gr_text "Night Shift Electronics"
+		(at 80.5 97 0)
 		(layer "F.SilkS")
 		(effects
@@
 	)
 	(via
+		(at 80 56.5)
+		(size 0.6)
+		(drill 0.3)
+		(layers "F.Cu" "B.Cu")
+		(free yes)
+		(net "GND")
+	)
+	(via
 		(at 72.397262 71.948824)
 		(size 0.6)
@@
 	)
 	(via
+		(at 93.5 31.5)
+		(size 0.6)
+		(drill 0.3)
+		(layers "F.Cu" "B.Cu")
+		(free yes)
+		(net "GND")
+	)
+	(via
 		(at 46.5 45.075001)
 		(size 0.6)
@@
 	)
 	(via
+		(at 88.5 32)
+		(size 0.6)
+		(drill 0.3)
+		(layers "F.Cu" "B.Cu")
+		(free yes)
+		(net "GND")
+	)
+	(via
 		(at 65.25 53.025001)
 		(size 0.6)
@@
 		(net "GND")
 	)
+	(via
+		(at 88.5 34)
+		(size 0.6)
+		(drill 0.3)
+		(layers "F.Cu" "B.Cu")
+		(free yes)
+		(net "GND")
+	)
